Commit message: Added d415 camera for gazebo and set gazebo paths

File: realsense2_description/urdf/_d415.urdf.xacro (robot description, xacro)
@@ -1,3 +1,3 @@
-<?xml version="1.0"?>
+<?xml version="1.0" ?>
 <!--
 License: Apache 2.0. See LICENSE file in root directory.
@@ -7,51 +7,53 @@
 -->
 <robot name="sensor_d415" xmlns:xacro="http://ros.org/wiki/xacro">
+  <!--File includes-->
+  <xacro:include filename="$(find realsense2_description)/urdf/_d415.gazebo.xacro" />
   <xacro:macro name="sensor_d415" params="name:=camera parent *origin">
     <xacro:property name="M_PI" value="3.1415926535897931" />
     <!-- The following values are approximate, and the camera node
      publishing TF values with actual calibrated camera extrinsic values -->
-    <xacro:property name="d415_cam_depth_to_left_ir_offset" value="0.0"/>
-    <xacro:property name="d415_cam_depth_to_right_ir_offset" value="-0.055"/>
-    <xacro:property name="d415_cam_depth_to_color_offset" value="0.015"/>
+    <xacro:property name="d415_cam_depth_to_left_ir_offset" value="0.0" />
+    <xacro:property name="d415_cam_depth_to_right_ir_offset" value="-0.055" />
+    <xacro:property name="d415_cam_depth_to_color_offset" value="0.015" />
     <!-- The following values model the aluminum peripherial case for the
   	d415 camera, with the camera joint represented by the actual
   	peripherial camera tripod mount -->
-    <xacro:property name="d415_cam_width" value="0.099"/>
-    <xacro:property name="d415_cam_height" value="0.023"/>
-    <xacro:property name="d415_cam_depth" value="0.02005"/>
-    <xacro:property name="d415_cam_mount_from_center_offset" value="0.00987"/>
+    <xacro:property name="d415_cam_width" value="0.099" />
+    <xacro:property name="d415_cam_height" value="0.023" />
+    <xacro:property name="d415_cam_depth" value="0.02005" />
+    <xacro:property name="d415_cam_mount_from_center_offset" value="0.00987" />
     <!-- The following offset is relative the the physical d415 camera peripherial
   	camera tripod mount -->
-    <xacro:property name="d415_cam_depth_px" value="${d415_cam_mount_from_center_offset}"/>
-    <xacro:property name="d415_cam_depth_py" value="0.020"/>
-    <xacro:property name="d415_cam_depth_pz" value="${d415_cam_height/2}"/>
+    <xacro:property name="d415_cam_depth_px" value="${d415_cam_mount_from_center_offset}" />
+    <xacro:property name="d415_cam_depth_py" value="0.020" />
+    <xacro:property name="d415_cam_depth_pz" value="${d415_cam_height/2}" />
     <material name="${name}_aluminum">
-	     <color rgba="0.5 0.5 0.5 1"/>
+      <color rgba="0.5 0.5 0.5 1" />
     </material>
     <!-- camera body, with origin at bottom screw mount -->
     <joint name="${name}_joint" type="fixed">
       <xacro:insert_block name="origin" />
-      <parent link="${parent}"/>
+      <parent link="${parent}" />
       <child link="${name}_bottom_screw_frame" />
     </joint>
-    <link name="${name}_bottom_screw_frame"/>
+    <link name="${name}_bottom_screw_frame" />
     <joint name="${name}_link_joint" type="fixed">
-      <origin xyz="0 ${d415_cam_depth_py} ${d415_cam_depth_pz}" rpy="0 0 0"/>
-      <parent link="${name}_bottom_screw_frame"/>
+      <origin xyz="0 ${d415_cam_depth_py} ${d415_cam_depth_pz}" rpy="0 0 0" />
+      <parent link="${name}_bottom_screw_frame" />
       <child link="${name}_link" />
     </joint>
     <link name="${name}_link">
       <visual>
-      <origin xyz="${d415_cam_mount_from_center_offset} ${-d415_cam_depth_py} 0" rpy="${M_PI/2} 0 ${M_PI/2}"/>
+        <origin xyz="${d415_cam_mount_from_center_offset} ${-d415_cam_depth_py} 0" rpy="${M_PI/2} 0 ${M_PI/2}" />
         <geometry>
           <!-- <box size="${d415_cam_width} ${d415_cam_height} ${d415_cam_depth}"/> -->
-	         <mesh filename="package://realsense2_description/meshes/d415.stl" />
+          <mesh filename="package://realsense2_description/meshes/d415.stl" />
         </geometry>
-        <material name="${name}_aluminum"/>
+        <material name="${name}_aluminum" />
       </visual>
       <collision>
-        <origin xyz="0 ${-d415_cam_depth_py} 0" rpy="0 0 0"/>
+        <origin xyz="0 ${-d415_cam_depth_py} 0" rpy="0 0 0" />
         <geometry>
-        <box size="${d415_cam_depth} ${d415_cam_width} ${d415_cam_height}"/>
+          <box size="${d415_cam_depth} ${d415_cam_width} ${d415_cam_height}" />
         </geometry>
       </collision>
@@ -65,9 +67,9 @@
     <!-- camera depth joints and links -->
     <joint name="${name}_depth_joint" type="fixed">
-      <origin xyz="0 0 0" rpy="0 0 0"/>
-      <parent link="${name}_link"/>
+      <origin xyz="0 0 0" rpy="0 0 0" />
+      <parent link="${name}_link" />
       <child link="${name}_depth_frame" />
     </joint>
-    <link name="${name}_depth_frame"/>
+    <link name="${name}_depth_frame" />
     <joint name="${name}_depth_optical_joint" type="fixed">
       <origin xyz="0 0 0" rpy="${-M_PI/2} 0 ${-M_PI/2}" />
@@ -75,5 +77,5 @@
       <child link="${name}_depth_optical_frame" />
     </joint>
-    <link name="${name}_depth_optical_frame"/>
+    <link name="${name}_depth_optical_frame" />
     <!-- camera left IR joints and links -->
     <joint name="${name}_left_ir_joint" type="fixed">
@@ -82,5 +84,5 @@
       <child link="${name}_left_ir_frame" />
     </joint>
-    <link name="${name}_left_ir_frame"/>
+    <link name="${name}_left_ir_frame" />
     <joint name="${name}_left_ir_optical_joint" type="fixed">
       <origin xyz="0 0 0" rpy="${-M_PI/2} 0 ${-M_PI/2}" />
@@ -88,5 +90,5 @@
       <child link="${name}_left_ir_optical_frame" />
     </joint>
-    <link name="${name}_left_ir_optical_frame"/>
+    <link name="${name}_left_ir_optical_frame" />
     <!-- camera right IR joints and links -->
     <joint name="${name}_right_ir_joint" type="fixed">
@@ -95,5 +97,5 @@
       <child link="${name}_right_ir_frame" />
     </joint>
-    <link name="${name}_right_ir_frame"/>
+    <link name="${name}_right_ir_frame" />
     <joint name="${name}_right_ir_optical_joint" type="fixed">
       <origin xyz="0 0 0" rpy="${-M_PI/2} 0 ${-M_PI/2}" />
@@ -101,5 +103,5 @@
       <child link="${name}_right_ir_optical_frame" />
     </joint>
-    <link name="${name}_right_ir_optical_frame"/>
+    <link name="${name}_right_ir_optical_frame" />
     <!-- camera color joints and links -->
     <joint name="${name}_color_joint" type="fixed">
@@ -108,5 +110,5 @@
       <child link="${name}_color_frame" />
     </joint>
-    <link name="${name}_color_frame"/>
+    <link name="${name}_color_frame" />
     <joint name="${name}_color_optical_joint" type="fixed">
       <origin xyz="0 0 0" rpy="${-M_PI/2} 0 ${-M_PI/2}" />
@@ -114,5 +116,7 @@
       <child link="${name}_color_optical_frame" />
     </joint>
-    <link name="${name}_color_optical_frame"/>
+    <link name="${name}_color_optical_frame" />
+    <!-- Realsense Gazebo Plugin -->
+    <xacro:gazebo_d415 camera_name="${name}" reference_link="${name}_link" topics_ns="${topics_ns}" depth_optical_frame="${name}_depth_optical_frame" color_optical_frame="${name}_color_optical_frame" infrared1_optical_frame="${name}_left_ir_optical_frame" infrared2_optical_frame="${name}_right_ir_optical_frame" publish_pointcloud="${publish_pointcloud}"/>
   </xacro:macro>
 </robot>

Commit message: fixed paths

File: realsense2_description/urdf/_d415.urdf.xacro (robot description, xacro)
@@ -48,5 +48,5 @@
         <geometry>
           <!-- <box size="${d415_cam_width} ${d415_cam_height} ${d415_cam_depth}"/> -->
-          <mesh filename="package://realsense2_description/meshes/d415.stl" />
+          <mesh filename="file://$(find realsense2_description)/meshes/d415.stl" />
         </geometry>
         <material name="${name}_aluminum" />

File: realsense2_description/urdf/_d435.urdf.xacro (robot description, xacro)
@@ -48,5 +48,5 @@
         <geometry>
           <!-- <box size="${d435_cam_width} ${d435_cam_height} ${d435_cam_depth}"/> -->
-          <mesh filename="package://realsense2_description/meshes/d435.dae" />
+          <mesh filename="file://$(find realsense2_description)/meshes/d435.dae" />
           <!--<mesh filename="package://realsense2_description/meshes/d435/d435.dae" />-->
         </geometry>

File: realsense_models/urdf/rs_d415_camera.urdf (robot description, URDF)
Before this commit: robot realsense2_camera, 11 links, 10 joints
Links:
- link rs_d415_link: geometry collision box size=0.02005 0.099 0.023; visual mesh filename=file:///home/developer/workspace/catkin_ws/src/ail/realsens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

File: realsense_models/urdf/rs_d435_camera.urdf (robot description, URDF)
Before this commit: robot realsense2_camera, 11 links, 10 joints
Links:
- link rs_d435_camera_link: geometry collision box size=0.02505 0.09 0.025; visual mesh filename=file:///home/developer/workspace/catkin_ws/src/ail/realsens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
