Commit message: Fixed xacro warnings

File: realsense2_description/urdf/_d415.gazebo.xacro (robot description, xacro)
@@ -1,3 +1,3 @@
-<?xml version="1.0"?>
+<?xml version="1.0" ?>
 <!--
 License: Apache 2.0. See LICENSE file in root directory.
@@ -6,5 +6,5 @@
 -->
 <robot xmlns:xacro="http://ros.org/wiki/xacro">
-  <xacro:macro name="gazebo_d415" params="camera_name reference_link topics_ns depth_optical_frame color_optical_frame infrared1_optical_frame infrared2_optical_frame publish_pointcloud:=true" >
+  <xacro:macro name="gazebo_d415" params="camera_name reference_link topics_ns depth_optical_frame color_optical_frame infrared1_optical_frame infrared2_optical_frame publish_pointcloud:=true">
     <!-- Load parameters to model's main link-->
     <xacro:property name="deg_to_rad" value="0.01745329251994329577" />

File: realsense2_description/urdf/_d415.urdf.xacro (robot description, xacro)
@@ -9,5 +9,5 @@
   <!--File includes-->
   <xacro:include filename="$(find realsense2_description)/urdf/_d415.gazebo.xacro" />
-  <xacro:macro name="sensor_d415" params="name:=camera parent *origin">
+  <xacro:macro name="sensor_d415" params="name:=rs_d415 topics_ns:=rs_d415 parent *origin publish_pointcloud:=true">
     <xacro:property name="M_PI" value="3.1415926535897931" />
     <!-- The following values are approximate, and the camera node
@@ -60,5 +60,5 @@
       <inertial>
         <!-- The following are not reliable values, and should not be used for modeling -->
-        <mass value="0.564" />
+        <mass value="0.072" />
         <origin xyz="0 0 0" />
         <inertia ixx="0.003881243" ixy="0.0" ixz="0.0" iyy="0.000498940" iyz="0.0" izz="0.003879257" />
@@ -118,5 +118,5 @@
     <link name="${name}_color_optical_frame" />
     <!-- Realsense Gazebo Plugin -->
-    <xacro:gazebo_d415 camera_name="${name}" reference_link="${name}_link" topics_ns="${topics_ns}" depth_optical_frame="${name}_depth_optical_frame" color_optical_frame="${name}_color_optical_frame" infrared1_optical_frame="${name}_left_ir_optical_frame" infrared2_optical_frame="${name}_right_ir_optical_frame" publish_pointcloud="${publish_pointcloud}"/>
+    <xacro:gazebo_d415 camera_name="${name}" reference_link="${name}_link" topics_ns="${topics_ns}" depth_optical_frame="${name}_depth_optical_frame" color_optical_frame="${name}_color_optical_frame" infrared1_optical_frame="${name}_left_ir_optical_frame" infrared2_optical_frame="${name}_right_ir_optical_frame" publish_pointcloud="${publish_pointcloud}" />
   </xacro:macro>
 </robot>

File: realsense2_description/urdf/_d435.gazebo.xacro (robot description, xacro)
@@ -1,3 +1,3 @@
-<?xml version="1.0"?>
+<?xml version="1.0" ?>
 <!--
 License: Apache 2.0. See LICENSE file in root directory.
@@ -6,5 +6,5 @@
 -->
 <robot xmlns:xacro="http://ros.org/wiki/xacro">
-  <xacro:macro name="gazebo_d435" params="camera_name reference_link topics_ns depth_optical_frame color_optical_frame infrared1_optical_frame infrared2_optical_frame publish_pointcloud:=true" >
+  <xacro:macro name="gazebo_d435" params="camera_name reference_link topics_ns depth_optical_frame color_optical_frame infrared1_optical_frame infrared2_optical_frame publish_pointcloud:=true">
     <!-- Load parameters to model's main link-->
     <xacro:property name="deg_to_rad" value="0.01745329251994329577" />
@@ -25,5 +25,5 @@
       <sensor name="${camera_name}color" type="camera">
         <camera name="${camera_name}">
-          <horizontal_fov>${69.4*deg_to_rad}</horizontal_fov>
+          <horizontal_fov>${69.0*deg_to_rad}</horizontal_fov>
           <image>
             <width>1920</width>
@@ -47,5 +47,5 @@
       <sensor name="${camera_name}ired1" type="camera">
         <camera name="${camera_name}">
-          <horizontal_fov>${85.2*deg_to_rad}</horizontal_fov>
+          <horizontal_fov>${87.0*deg_to_rad}</horizontal_fov>
           <image>
             <width>1280</width>
@@ -54,6 +54,6 @@
           </image>
           <clip>
-            <near>0.1</near>
-            <far>100</far>
+            <near>0.105</near>
+            <far>10</far>
           </clip>
           <noise>
@@ -69,5 +69,5 @@
       <sensor name="${camera_name}ired2" type="camera">
         <camera name="${camera_name}">
-          <horizontal_fov>${85.2*deg_to_rad}</horizontal_fov>
+          <horizontal_fov>${87.0*deg_to_rad}</horizontal_fov>
           <image>
             <width>1280</width>
@@ -76,6 +76,6 @@
           </image>
           <clip>
-            <near>0.1</near>
-            <far>100</far>
+            <near>0.105</near>
+            <far>10</far>
           </clip>
           <noise>

File: realsense2_description/urdf/_d435.urdf.xacro (robot description, xacro)
@@ -1,3 +1,3 @@
-<?xml version="1.0"?>
+<?xml version="1.0" ?>
 <!--
 License: Apache 2.0. See LICENSE file in root directory.
@@ -8,42 +8,42 @@
 <robot name="sensor_d435" xmlns:xacro="http://ros.org/wiki/xacro">
   <!--File includes-->
-  <xacro:include filename="$(find realsense2_description)/urdf/_d435.gazebo.xacro"/>
-  <xacro:macro name="sensor_d435" params="name:=camera topics_ns:=camera parent *origin publish_pointcloud:=true">
+  <xacro:include filename="$(find realsense2_description)/urdf/_d435.gazebo.xacro" />
+  <xacro:macro name="sensor_d435" params="name:=rs_d435_camera topics_ns:=rs_d435_camera parent *origin publish_pointcloud:=true">
     <xacro:property name="M_PI" value="3.1415926535897931" />
     <!-- The following values are approximate, and the camera node
      publishing TF values with actual calibrated camera extrinsic values -->
-    <xacro:property name="d435_cam_depth_to_left_ir_offset" value="0.0"/>
-    <xacro:property name="d435_cam_depth_to_right_ir_offset" value="-0.050"/>
-    <xacro:property name="d435_cam_depth_to_color_offset" value="0.015"/>
+    <xacro:property name="d435_cam_depth_to_left_ir_offset" value="0.0" />
+    <xacro:property name="d435_cam_depth_to_right_ir_offset" value="-0.050" />
+    <xacro:property name="d435_cam_depth_to_color_offset" value="0.015" />
     <!-- The following values model the aluminum peripherial case for the
     D435 camera, with the camera joint represented by the actual
     peripherial camera tripod mount -->
-    <xacro:property name="d435_cam_width" value="0.090"/>
-    <xacro:property name="d435_cam_height" value="0.025"/>
-    <xacro:property name="d435_cam_depth" value="0.02505"/>
-    <xacro:property name="d435_cam_mount_from_center_offset" value="0.0149"/>
+    <xacro:property name="d435_cam_width" value="0.090" />
+    <xacro:property name="d435_cam_height" value="0.025" />
+    <xacro:property name="d435_cam_depth" value="0.02505" />
+    <xacro:property name="d435_cam_mount_from_center_offset" value="0.0149" />
     <!-- The following offset is relative the the physical D435 camera peripherial
     camera tripod mount -->
-    <xacro:property name="d435_cam_depth_px" value="${d435_cam_mount_from_center_offset}"/>
-    <xacro:property name="d435_cam_depth_py" value="0.0175"/>
-    <xacro:property name="d435_cam_depth_pz" value="${d435_cam_height/2}"/>
+    <xacro:property name="d435_cam_depth_px" value="${d435_cam_mount_from_center_offset}" />
+    <xacro:property name="d435_cam_depth_py" value="0.0175" />
+    <xacro:property name="d435_cam_depth_pz" value="${d435_cam_height/2}" />
     <material name="${name}_aluminum">
-    <color rgba="0.5 0.5 0.5 1"/>
+      <color rgba="0.5 0.5 0.5 1" />
     </material>
     <!-- camera body, with origin at bottom screw mount -->
     <joint name="${name}_joint" type="fixed">
       <xacro:insert_block name="origin" />
-      <parent link="${parent}"/>
+      <parent link="${parent}" />
       <child link="${name}_bottom_screw_frame" />
     </joint>
-    <link name="${name}_bottom_screw_frame"/>
+    <link name="${name}_bottom_screw_frame" />
     <joint name="${name}_link_joint" type="fixed">
-      <origin xyz="0 ${d435_cam_depth_py} ${d435_cam_depth_pz}" rpy="0 0 0"/>
-      <parent link="${name}_bottom_screw_frame"/>
+      <origin xyz="0 ${d435_cam_depth_py} ${d435_cam_depth_pz}" rpy="0 0 0" />
+      <parent link="${name}_bottom_screw_frame" />
       <child link="${name}_link" />
     </joint>
     <link name="${name}_link">
       <visual>
-      <origin xyz="${d435_cam_mount_from_center_offset} ${-d435_cam_depth_py} 0" rpy="${M_PI/2} 0 ${M_PI/2}"/>
+        <origin xyz="${d435_cam_mount_from_center_offset} ${-d435_cam_depth_py} 0" rpy="${M_PI/2} 0 ${M_PI/2}" />
         <geometry>
           <!-- <box size="${d435_cam_width} ${d435_cam_height} ${d435_cam_depth}"/> -->
@@ -51,15 +51,15 @@
           <!--<mesh filename="package://realsense2_description/meshes/d435/d435.dae" />-->
         </geometry>
-        <material name="${name}_aluminum"/>
+        <material name="${name}_aluminum" />
       </visual>
       <collision>
-        <origin xyz="0 ${-d435_cam_depth_py} 0" rpy="0 0 0"/>
+        <origin xyz="0 ${-d435_cam_depth_py} 0" rpy="0 0 0" />
         <geometry>
-        <box size="${d435_cam_depth} ${d435_cam_width} ${d435_cam_height}"/>
+          <box size="${d435_cam_depth} ${d435_cam_width} ${d435_cam_height}" />
         </geometry>
       </collision>
       <inertial>
         <!-- The following are not reliable values, and should not be used for modeling -->
-        <mass value="0.564" />
+        <mass value="0.072" />
         <origin xyz="0 0 0" />
         <inertia ixx="0.003881243" ixy="0.0" ixz="0.0" iyy="0.000498940" iyz="0.0" izz="0.003879257" />
@@ -68,9 +68,9 @@
     <!-- camera depth joints and links -->
     <joint name="${name}_depth_joint" type="fixed">
-      <origin xyz="0 0 0" rpy="0 0 0"/>
-      <parent link="${name}_link"/>
+      <origin xyz="0 0 0" rpy="0 0 0" />
+      <parent link="${name}_link" />
       <child link="${name}_depth_frame" />
     </joint>
-    <link name="${name}_depth_frame"/>
+    <link name="${name}_depth_frame" />
     <joint name="${name}_depth_optical_joint" type="fixed">
       <origin xyz="0 0 0" rpy="${-M_PI/2} 0 ${-M_PI/2}" />
@@ -78,5 +78,5 @@
       <child link="${name}_depth_optical_frame" />
     </joint>
-    <link name="${name}_depth_optical_frame"/>
+    <link name="${name}_depth_optical_frame" />
     <!-- camera left IR joints and links -->
     <joint name="${name}_left_ir_joint" type="fixed">
@@ -85,5 +85,5 @@
       <child link="${name}_left_ir_frame" />
     </joint>
-    <link name="${name}_left_ir_frame"/>
+    <link name="${name}_left_ir_frame" />
     <joint name="${name}_left_ir_optical_joint" type="fixed">
       <origin xyz="0 0 0" rpy="${-M_PI/2} 0 ${-M_PI/2}" />
@@ -91,5 +91,5 @@
       <child link="${name}_left_ir_optical_frame" />
     </joint>
-    <link name="${name}_left_ir_optical_frame"/>
+    <link name="${name}_left_ir_optical_frame" />
     <!-- camera right IR joints and links -->
     <joint name="${name}_right_ir_joint" type="fixed">
@@ -98,5 +98,5 @@
       <child link="${name}_right_ir_frame" />
     </joint>
-    <link name="${name}_right_ir_frame"/>
+    <link name="${name}_right_ir_frame" />
     <joint name="${name}_right_ir_optical_joint" type="fixed">
       <origin xyz="0 0 0" rpy="${-M_PI/2} 0 ${-M_PI/2}" />
@@ -104,5 +104,5 @@
       <child link="${name}_right_ir_optical_frame" />
     </joint>
-    <link name="${name}_right_ir_optical_frame"/>
+    <link name="${name}_right_ir_optical_frame" />
     <!-- camera color joints and links -->
     <joint name="${name}_color_joint" type="fixed">
@@ -111,5 +111,5 @@
       <child link="${name}_color_frame" />
     </joint>
-    <link name="${name}_color_frame"/>
+    <link name="${name}_color_frame" />
     <joint name="${name}_color_optical_joint" type="fixed">
       <origin xyz="0 0 0" rpy="${-M_PI/2} 0 ${-M_PI/2}" />
@@ -117,7 +117,7 @@
       <child link="${name}_color_optical_frame" />
     </joint>
-    <link name="${name}_color_optical_frame"/>
+    <link name="${name}_color_optical_frame" />
     <!-- Realsense Gazebo Plugin -->
-    <xacro:gazebo_d435 camera_name="${name}" reference_link="${name}_link" topics_ns="${topics_ns}" depth_optical_frame="${name}_depth_optical_frame" color_optical_frame="${name}_color_optical_frame" infrared1_optical_frame="${name}_left_ir_optical_frame" infrared2_optical_frame="${name}_right_ir_optical_frame" publish_pointcloud="${publish_pointcloud}"/>
+    <xacro:gazebo_d435 camera_name="${name}" reference_link="${name}_link" topics_ns="${topics_ns}" depth_optical_frame="${name}_depth_optical_frame" color_optical_frame="${name}_color_optical_frame" infrared1_optical_frame="${name}_left_ir_optical_frame" infrared2_optical_frame="${name}_right_ir_optical_frame" publish_pointcloud="${publish_pointcloud}" />
   </xacro:macro>
 </robot>

File: realsense2_description/urdf/test_d415_camera.urdf.xacro (robot description, xacro)
@@ -3,6 +3,6 @@
   <xacro:include filename="$(find realsense2_description)/urdf/_d415.urdf.xacro" />
   <link name="base_link" />
-  <sensor_d415 parent="base_link">
+  <xacro:sensor_d415 parent="base_link">
     <origin xyz="0 0 0" rpy="0 0 0"/>
-  </sensor_d415>
+  </xacro:sensor_d415>
 </robot>

File: realsense2_description/urdf/test_d435_camera.urdf.xacro (robot description, xacro)
@@ -3,6 +3,6 @@
   <xacro:include filename="$(find realsense2_description)/urdf/_d435.urdf.xacro" />
   <link name="base_link" />
-  <sensor_d435 parent="base_link">
+  <xacro:sensor_d435 parent="base_link">
     <origin xyz="0 0 0" rpy="0 0 0"/>
-  </sensor_d435>
+  </xacro:sensor_d435>
 </robot>
