Commit message: added option to set frame rate

File: realsense2_description/urdf/_d415.gazebo.xacro (robot description, xacro)
@@ -6,5 +6,5 @@
 -->
 <robot xmlns:xacro="http://ros.org/wiki/xacro">
-  <xacro:macro name="gazebo_d415" params="camera_name reference_link topics_ns depth_optical_frame color_optical_frame infrared1_optical_frame infrared2_optical_frame color_width:=1920 color_height:=1080 depth_width:=1280 depth_height:=720 disable_color:=false disable_depth:=false disable_ired:=true publish_pointcloud:=true">
+  <xacro:macro name="gazebo_d415" params="camera_name reference_link topics_ns depth_optical_frame color_optical_frame infrared1_optical_frame infrared2_optical_frame color_width:=1920 color_height:=1080 depth_width:=1280 depth_height:=720 disable_color:=false disable_depth:=false disable_ired:=true publish_pointcloud:=true update_rate:=30">
     <!-- Load parameters to model's main link-->
     <xacro:property name="deg_to_rad" value="0.01745329251994329577" />
@@ -43,5 +43,5 @@
           </camera>
           <always_on>1</always_on>
-          <update_rate>30</update_rate>
+          <update_rate>${update_rate}</update_rate>
           <visualize>1</visualize>
         </sensor>
@@ -67,5 +67,5 @@
           </camera>
           <always_on>1</always_on>
-          <update_rate>90</update_rate>
+          <update_rate>${update_rate}</update_rate>
           <visualize>0</visualize>
         </sensor>
@@ -89,5 +89,5 @@
           </camera>
           <always_on>1</always_on>
-          <update_rate>90</update_rate>
+          <update_rate>${update_rate}</update_rate>
           <visualize>0</visualize>
         </sensor>
@@ -112,5 +112,5 @@
           </camera>
           <always_on>1</always_on>
-          <update_rate>90</update_rate>
+          <update_rate>${update_rate}</update_rate>
           <visualize>0</visualize>
         </sensor>
@@ -123,7 +123,7 @@
         <disableDepth>${disable_depth}</disableDepth>
         <disableIred>${disable_ired}</disableIred>
-        <depthUpdateRate>60.0</depthUpdateRate>
-        <colorUpdateRate>60.0</colorUpdateRate>
-        <infraredUpdateRate>60.0</infraredUpdateRate>
+        <depthUpdateRate>${update_rate}</depthUpdateRate>
+        <colorUpdateRate>${update_rate}</colorUpdateRate>
+        <infraredUpdateRate>${update_rate}</infraredUpdateRate>
         <depthTopicName>depth/color/image_raw</depthTopicName>
         <depthCameraInfoTopicName>depth/color/camera_info</depthCameraInfoTopicName>

File: realsense2_description/urdf/_d415.urdf.xacro (robot description, xacro)
@@ -9,5 +9,5 @@
   <!--File includes-->
   <xacro:include filename="$(find realsense2_description)/urdf/_d415.gazebo.xacro" />
-  <xacro:macro name="sensor_d415" params="name:=camera_rs_d415 topics_ns:=camera_rs_d415 parent *origin color_width:=1920 color_height:=1080 depth_width:=1280 depth_height:=720 disable_color:=false disable_depth:=false disable_ired:=true publish_pointcloud:=true">
+  <xacro:macro name="sensor_d415" params="name:=camera_rs_d415 topics_ns:=camera_rs_d415 parent *origin color_width:=1920 color_height:=1080 depth_width:=1280 depth_height:=720 disable_color:=false disable_depth:=false disable_ired:=true publish_pointcloud:=true update_rate:=30">
     <xacro:property name="M_PI" value="3.1415926535897931" />
     <!-- The following values are approximate, and the camera node
@@ -118,5 +118,5 @@
     <link name="${name}_color_optical_frame" />
     <!-- Realsense Gazebo Plugin -->
-    <xacro:gazebo_d415 camera_name="${name}" reference_link="${name}_link" topics_ns="${topics_ns}" depth_optical_frame="${name}_depth_optical_frame" color_optical_frame="${name}_color_optical_frame" infrared1_optical_frame="${name}_left_ir_optical_frame" infrared2_optical_frame="${name}_right_ir_optical_frame" color_width="${color_width}" color_height="${color_height}" depth_width="${depth_width}" depth_height="${depth_height}" disable_color="${disable_color}" disable_depth="${disable_depth}" disable_ired="${disable_ired}" publish_pointcloud="${publish_pointcloud}" />
+    <xacro:gazebo_d415 camera_name="${name}" reference_link="${name}_link" topics_ns="${topics_ns}" depth_optical_frame="${name}_depth_optical_frame" color_optical_frame="${name}_color_optical_frame" infrared1_optical_frame="${name}_left_ir_optical_frame" infrared2_optical_frame="${name}_right_ir_optical_frame" color_width="${color_width}" color_height="${color_height}" depth_width="${depth_width}" depth_height="${depth_height}" disable_color="${disable_color}" disable_depth="${disable_depth}" disable_ired="${disable_ired}" publish_pointcloud="${publish_pointcloud}" update_rate="${update_rate}" />
   </xacro:macro>
 </robot>

File: realsense2_description/urdf/_d435.gazebo.xacro (robot description, xacro)
@@ -6,5 +6,5 @@
 -->
 <robot xmlns:xacro="http://ros.org/wiki/xacro">
-  <xacro:macro name="gazebo_d435" params="camera_name reference_link topics_ns depth_optical_frame color_optical_frame infrared1_optical_frame infrared2_optical_frame color_width:=1920 color_height:=1080 depth_width:=1280 depth_height:=720 disable_color:=false disable_depth:=false disable_ired:=true publish_pointcloud:=true">
+  <xacro:macro name="gazebo_d435" params="camera_name reference_link topics_ns depth_optical_frame color_optical_frame infrared1_optical_frame infrared2_optical_frame color_width:=1920 color_height:=1080 depth_width:=1280 depth_height:=720 disable_color:=false disable_depth:=false disable_ired:=true publish_pointcloud:=true update_rate:=30">
     <!-- Load parameters to model's main link-->
     <xacro:property name="deg_to_rad" value="0.01745329251994329577" />
@@ -43,5 +43,5 @@
           </camera>
           <always_on>1</always_on>
-          <update_rate>30</update_rate>
+          <update_rate>${update_rate}</update_rate>
           <visualize>1</visualize>
         </sensor>
@@ -67,5 +67,5 @@
           </camera>
           <always_on>1</always_on>
-          <update_rate>90</update_rate>
+          <update_rate>${update_rate}</update_rate>
           <visualize>0</visualize>
         </sensor>
@@ -89,5 +89,5 @@
           </camera>
           <always_on>1</always_on>
-          <update_rate>90</update_rate>
+          <update_rate>${update_rate}</update_rate>
           <visualize>0</visualize>
         </sensor>
@@ -112,5 +112,5 @@
           </camera>
           <always_on>1</always_on>
-          <update_rate>90</update_rate>
+          <update_rate>${update_rate}</update_rate>
           <visualize>0</visualize>
         </sensor>
@@ -123,7 +123,7 @@
         <disableDepth>${disable_depth}</disableDepth>
         <disableIred>${disable_ired}</disableIred>
-        <depthUpdateRate>60.0</depthUpdateRate>
-        <colorUpdateRate>60.0</colorUpdateRate>
-        <infraredUpdateRate>60.0</infraredUpdateRate>
+        <depthUpdateRate>${update_rate}</depthUpdateRate>
+        <colorUpdateRate>${update_rate}</colorUpdateRate>
+        <infraredUpdateRate>${update_rate}</infraredUpdateRate>
         <depthTopicName>depth/color/image_raw</depthTopicName>
         <depthCameraInfoTopicName>depth/color/camera_info</depthCameraInfoTopicName>

File: realsense2_description/urdf/_d435.urdf.xacro (robot description, xacro)
@@ -9,5 +9,5 @@
   <!--File includes-->
   <xacro:include filename="$(find realsense2_description)/urdf/_d435.gazebo.xacro" />
-  <xacro:macro name="sensor_d435" params="name:=camera_rs_d435 topics_ns:=camera_rs_d435 parent *origin color_width:=1920 color_height:=1080 depth_width:=1280 depth_height:=720 disable_color:=false disable_depth:=false disable_ired:=true publish_pointcloud:=true">
+  <xacro:macro name="sensor_d435" params="name:=camera_rs_d435 topics_ns:=camera_rs_d435 parent *origin color_width:=1920 color_height:=1080 depth_width:=1280 depth_height:=720 disable_color:=false disable_depth:=false disable_ired:=true publish_pointcloud:=true update_rate:=30">
     <xacro:property name="M_PI" value="3.1415926535897931" />
     <!-- The following values are approximate, and the camera node
@@ -119,5 +119,5 @@
     <link name="${name}_color_optical_frame" />
     <!-- Realsense Gazebo Plugin -->
-    <xacro:gazebo_d435 camera_name="${name}" reference_link="${name}_link" topics_ns="${topics_ns}" depth_optical_frame="${name}_depth_optical_frame" color_optical_frame="${name}_color_optical_frame" infrared1_optical_frame="${name}_left_ir_optical_frame" infrared2_optical_frame="${name}_right_ir_optical_frame" color_width="${color_width}" color_height="${color_height}" depth_width="${depth_width}" depth_height="${depth_height}" disable_color="${disable_color}" disable_depth="${disable_depth}" disable_ired="${disable_ired}" publish_pointcloud="${publish_pointcloud}" />
+    <xacro:gazebo_d435 camera_name="${name}" reference_link="${name}_link" topics_ns="${topics_ns}" depth_optical_frame="${name}_depth_optical_frame" color_optical_frame="${name}_color_optical_frame" infrared1_optical_frame="${name}_left_ir_optical_frame" infrared2_optical_frame="${name}_right_ir_optical_frame" color_width="${color_width}" color_height="${color_height}" depth_width="${depth_width}" depth_height="${depth_height}" disable_color="${disable_color}" disable_depth="${disable_depth}" disable_ired="${disable_ired}" publish_pointcloud="${publish_pointcloud}" update_rate="${update_rate}" />
   </xacro:macro>
 </robot>
